File: schematic/keypad/keypad.kicad_pcb (KiCad board)
At the start: 2 copper layers, 95 x 100 mm, 13 parts, among them J1 Capacitive Touch Buttons, SW1 SW_Push, SW2 SW_Push, SW3 SW_Push, SW4 RotaryEncoder_Switch_MP, SW5 RotaryEncoder_Switch_MP, U1 Waveshare ESP32-S3-ZERO

Commit message: removed logo on the PCB
Parts:
- moved G*** 2.00 mm to (173.5, 90.8)
Changed lines of the file:
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@@
 			(at 0 0 0)
 			(layer "F.SilkS")
+			(hide yes)
 			(effects
 				(font
@@
 	(footprint "LOGO"
 		(layer "B.Cu")
-		(at 175.5 90.75 -90)
+		(at 173.5 90.75 -90)
 		(property "Reference" "G***"
 			(at 0 0 90)
